Commit message: fix display.launch.py file

File: src/volcanibot_description/urdf/volcanibot_description.urdf (robot description, URDF)
Before this commit: robot volcanibot_description, 5 links, 4 joints
Links:
- link base_link: geometry collision mesh filename=package://volcanibot_description/meshes/base_link.STL; visual mesh filename=package://volcanibot_description/meshes/base_link.STL
- link link_BL: geometry collision mesh filename=package://volcanibot_description/meshes/link_BL.STL; visual mesh filename=package://volcanibot_description/meshes/link_BL.STL
- link link_BR: geometry collision mesh filename=package://volcanibot_description/meshes/link_BR.STL; visual mesh filename=package://volcanibot_description/meshes/link_BR.STL
- link link_FL: geometry collision mesh filename=package://volcanibot_description/meshes/link_FL.STL; visual mesh filename=package://volcanibot_description/meshes/link_FL.STL
- link link_FR: geometry collision mesh filename=package://volcanibot_description/meshes/link_FR.STL; visual mesh filename=package://volcanibot_description/meshes/link_FR.STL
