Commit message: Add bringup pkg, Roboteq hw interface, Ouster lidar + optional camera
- volcanibot_bringup: sim_bringup.launch.py + real_bringup.launch.py with
  shared lidar/camera/rviz args (defaults: lidar=false, camera=false,
  rviz=true). Sim default world is feild.
- volcanibot_hardware_interface: ros2_control SystemInterface plugin for
  the Roboteq dual-channel motor controller over serial; udev rule and
  auto-detecting install.sh that creates /dev/roboteq. Adapted from
  konu-droid/diffdrive_ros2_control (Apache-2.0).
- install_udev.sh: ws-root wrapper around the in-package udev installer.
- volcanibot_description: split ros2_control by use_sim (sim drives all 4
  wheels via gz_ros2_control, real drives only the rear pair via the
  Roboteq plugin); RGBD camera now gated behind a `camera` arg; new
  volcanibot_lidar.xacro for the Ouster Rev5 OS2, mounted ~0.6 m off the
  ground on the front of base_link; feild.sdf gets a full <gui> mirror of
  the default gui.config with a grey theme and a camera_pose aimed at the
  robot spawn.
- gazebo.launch.py: forwards lidar/camera xacro args; bridges /scan
  (LaserScan), /scan/points (PointCloud2), and /camera/* only when the
  matching sensor is enabled.
- controller configs: sim YAML keeps the 4-joint diff-drive layout;
  volcanibot_controllers_real.yaml drives only rear_*_wheel_joint.

Co-Authored-By: Claude Opus 4.7 (1M context) <noreply@anthropic.com>

File: src/volcanibot_description/urdf/volcanibot.xacro (robot description, xacro)
@@ -2,4 +2,9 @@
 <robot xmlns:xacro="http://www.ros.org/wiki/xacro" name="volcanibot">
   <xacro:arg name="is_ignition" default="true" />
+  <xacro:arg name="use_sim" default="true" />
+  <xacro:arg name="lidar" default="false" />
+  <xacro:arg name="camera" default="false" />
+  <xacro:arg name="serial_port" default="/dev/roboteq" />
+  <xacro:arg name="baud_rate" default="115200" />
   <!-- Include Gazebo plugins -->
   <xacro:include filename="$(find volcanibot_description)/urdf/volcanibot_gazebo.xacro" />
@@ -8,4 +13,8 @@
   <!-- Colors -->
   <xacro:include filename="$(find volcanibot_description)/urdf/materials.xacro" />
+  <!-- Optional Ouster Rev5 (OS2) lidar -->
+  <xacro:if value="$(arg lidar)">
+    <xacro:include filename="$(find volcanibot_description)/urdf/volcanibot_lidar.xacro" />
+  </xacro:if>
   <!-- Define the world link -->
   <link name="base_footprint"/>
@@ -205,44 +214,45 @@
       xyz="0 1 0" />
   </joint>
-    <!-- Depth Camera -->
-  <joint type="fixed" name="camera_joint">
-    <origin xyz="0.6 0 0.07" rpy="0 0.2 0"/>
-    <child link="camera_link"/>
-    <parent link="base_link"/>
-    <axis xyz="0 1 0" />
-  </joint>
-  <link name='camera_link'>
-    <pose>0 0 0 0 0 0</pose>
-    <inertial>
-      <mass value="0.1"/>
-      <origin xyz="0 0 0" rpy="0 0 0"/>
-      <inertia
-          ixx="1e-6" ixy="0" ixz="0"
-          iyy="1e-6" iyz="0"
-          izz="1e-6"
-      />
-    </inertial>
-    <collision name='collision'>
-      <origin xyz="0 0 0" rpy="0 0 0"/>
-      <geometry>
-         <box size=".03 .03 .03"/>
-      </geometry>
-    </collision>
-    <visual name='camera_link_visual'>
-      <origin xyz="0 0 0" rpy="0 0 0"/>
-      <geometry>
-        <box size=".03 .03 .03"/>
-      </geometry>
-    </visual>
-  </link>
-  <gazebo reference="camera_link">
-    <material>Gazebo/Red</material>
-  </gazebo>
-  <joint type="fixed" name="camera_optical_joint">
-    <origin xyz="0 0 0" rpy="-1.5707 0 -1.5707"/>
-    <child link="camera_link_optical"/>
-    <parent link="camera_link"/>
-  </joint>
-  <link name="camera_link_optical">
-  </link>
+  <!-- Optional RGBD camera -->
+  <xacro:if value="$(arg camera)">
+    <joint type="fixed" name="camera_joint">
+      <origin xyz="0.6 0 0.07" rpy="0 0.2 0"/>
+      <child link="camera_link"/>
+      <parent link="base_link"/>
+      <axis xyz="0 1 0" />
+    </joint>
+    <link name="camera_link">
+      <inertial>
+        <mass value="0.1"/>
+        <origin xyz="0 0 0" rpy="0 0 0"/>
+        <inertia
+            ixx="1e-6" ixy="0" ixz="0"
+            iyy="1e-6" iyz="0"
+            izz="1e-6"
+        />
+      </inertial>
+      <collision>
+        <origin xyz="0 0 0" rpy="0 0 0"/>
+        <geometry>
+          <box size="0.03 0.03 0.03"/>
+        </geometry>
+      </collision>
+      <visual>
+        <origin xyz="0 0 0" rpy="0 0 0"/>
+        <geometry>
+          <box size="0.03 0.03 0.03"/>
+        </geometry>
+      </visual>
+    </link>
+    <gazebo reference="camera_link">
+      <material>Gazebo/Red</material>
+    </gazebo>
+    <joint type="fixed" name="camera_optical_joint">
+      <origin xyz="0 0 0" rpy="-1.5707 0 -1.5707"/>
+      <child link="camera_link_optical"/>
+      <parent link="camera_link"/>
+    </joint>
+    <link name="camera_link_optical">
+    </link>
+  </xacro:if>
 </robot>

File: src/volcanibot_description/urdf/volcanibot_gazebo.xacro (robot description, xacro)
@@ -38,39 +38,78 @@
     <fdir1>1 0 0</fdir1>
   </gazebo>
-  <!-- ROS 2 Control -->
-  <gazebo>
-    <!-- ROS 2 Humble -->
-    <xacro:if value="$(arg is_ignition)">
-      <plugin filename="ign_ros2_control-system" name="ign_ros2_control::IgnitionROS2ControlPlugin">
-        <parameters>$(find volcanibot_controller)/config/volcanibot_controllers.yaml</parameters>
-      </plugin>
-    </xacro:if>
-    <!-- ROS 2 Iron or above -->
-    <xacro:unless value="$(arg is_ignition)">
-      <plugin filename="gz_ros2_control-system" name="gz_ros2_control::GazeboSimROS2ControlPlugin">
-        <parameters>$(find volcanibot_controller)/config/volcanibot_controllers.yaml</parameters>
-      </plugin>
-    </xacro:unless>
-  </gazebo>
-  <gazebo reference="camera_link">
-    <sensor name="rgbd_camera" type="rgbd_camera">
-      <camera>
-        <horizontal_fov>1.25</horizontal_fov>
-        <image>
-          <width>320</width>
-          <height>240</height>
-        </image>
-        <clip>
-          <near>0.3</near>
-          <far>15</far>
-        </clip>
-        <optical_frame_id>camera_link_optical</optical_frame_id>
-      </camera>
-      <always_on>1</always_on>
-      <update_rate>20</update_rate>
-      <visualize>true</visualize>
-      <topic>camera</topic>
-      <gz_frame_id>camera_link</gz_frame_id>
-    </sensor>
-  </gazebo>
+  <!-- ROS 2 Control: Gazebo plugin loader, sim only -->
+  <xacro:if value="$(arg use_sim)">
+    <gazebo>
+      <!-- ROS 2 Humble -->
+      <xacro:if value="$(arg is_ignition)">
+        <plugin filename="ign_ros2_control-system" name="ign_ros2_control::IgnitionROS2ControlPlugin">
+          <parameters>$(find volcanibot_controller)/config/volcanibot_controllers.yaml</parameters>
+        </plugin>
+      </xacro:if>
+      <!-- ROS 2 Iron or above -->
+      <xacro:unless value="$(arg is_ignition)">
+        <plugin filename="gz_ros2_control-system" name="gz_ros2_control::GazeboSimROS2ControlPlugin">
+          <parameters>$(find volcanibot_controller)/config/volcanibot_controllers.yaml</parameters>
+        </plugin>
+      </xacro:unless>
+    </gazebo>
+  </xacro:if>
+  <!-- Optional RGBD camera sensor -->
+  <xacro:if value="$(arg camera)">
+    <gazebo reference="camera_link">
+      <sensor name="rgbd_camera" type="rgbd_camera">
+        <camera>
+          <horizontal_fov>1.25</horizontal_fov>
+          <image>
+            <width>320</width>
+            <height>240</height>
+          </image>
+          <clip>
+            <near>0.3</near>
+            <far>15</far>
+          </clip>
+          <optical_frame_id>camera_link_optical</optical_frame_id>
+        </camera>
+        <always_on>1</always_on>
+        <update_rate>20</update_rate>
+        <visualize>true</visualize>
+        <topic>camera</topic>
+        <gz_frame_id>camera_link</gz_frame_id>
+      </sensor>
+    </gazebo>
+  </xacro:if>
+  <!-- Optional Ouster Rev5 (OS2) lidar -->
+  <xacro:if value="$(arg lidar)">
+    <gazebo reference="os_sensor">
+      <sensor name="ouster_os2" type="gpu_lidar">
+        <pose>0 0 0.0435 0 0 0</pose>
+        <update_rate>10</update_rate>
+        <topic>scan</topic>
+        <gz_frame_id>os_lidar</gz_frame_id>
+        <ray>
+          <scan>
+            <horizontal>
+              <samples>1024</samples>
+              <resolution>1</resolution>
+              <min_angle>-3.14159</min_angle>
+              <max_angle>3.14159</max_angle>
+            </horizontal>
+            <vertical>
+              <samples>128</samples>
+              <resolution>1</resolution>
+              <min_angle>-0.19635</min_angle>
+              <max_angle>0.19635</max_angle>
+            </vertical>
+          </scan>
+          <range>
+            <min>0.4</min>
+            <max>240.0</max>
+            <resolution>0.03</resolution>
+          </range>
+        </ray>
+        <always_on>1</always_on>
+        <visualize>true</visualize>
+      </sensor>
+    </gazebo>
+  </xacro:if>
 </robot>

File: src/volcanibot_description/urdf/volcanibot_ros2_control.xacro (robot description, xacro)
@@ -2,50 +2,64 @@
 <robot xmlns:xacro="http://www.ros.org/wiki/xacro" name="volcanibot">
     <ros2_control name="RobotSystem" type="system">
-        <!-- ros2_control Gazebo -->
-        <!-- ROS 2 Humble -->
-        <xacro:if value="$(arg is_ignition)">
-            <hardware>
-                <plugin>ign_ros2_control/IgnitionSystem</plugin>
-            </hardware>
-        </xacro:if>
-        <!-- ROS 2 Iron or above -->
-        <xacro:unless value="$(arg is_ignition)">
-            <hardware>
-                <plugin>gz_ros2_control/GazeboSimSystem</plugin>
-            </hardware>
-        </xacro:unless>
-        <!-- ros2_control Common Interfaces -->
-        <joint name="rear_right_wheel_joint">
+        <hardware>
+            <xacro:if value="$(arg use_sim)">
+                <!-- ROS 2 Humble: Ignition Gazebo plugin -->
+                <xacro:if value="$(arg is_ignition)">
+                    <plugin>ign_ros2_control/IgnitionSystem</plugin>
+                </xacro:if>
+                <!-- ROS 2 Iron and above: gz Sim plugin -->
+                <xacro:unless value="$(arg is_ignition)">
+                    <plugin>gz_ros2_control/GazeboSimSystem</plugin>
+                </xacro:unless>
+            </xacro:if>
+            <xacro:unless value="$(arg use_sim)">
+                <plugin>volcanibot_hardware_interface/RoboteqDiffDriveSystem</plugin>
+                <param name="port">$(arg serial_port)</param>
+                <param name="baud_rate">$(arg baud_rate)</param>
+                <param name="timeout_ms">1000</param>
+                <param name="gear_ratio">1.0</param>
+                <param name="left_wheel_name">rear_left_wheel_joint</param>
+                <param name="right_wheel_name">rear_right_wheel_joint</param>
+            </xacro:unless>
+        </hardware>
+        <!-- In sim, all 4 wheels are independently controlled by Gazebo (the
+             physics engine doesn't support URDF mimic joints). On the real
+             robot only the rear wheels are motorized; the front wheels are
+             mechanically chained to the rear and so are not exposed to
+             ros2_control. -->
+        <joint name="rear_left_wheel_joint">
             <command_interface name="velocity">
-              <param name="min">-1</param>
-              <param name="max">1</param>
+              <param name="min">-10</param>
+              <param name="max">10</param>
             </command_interface>
             <state_interface name="position" />
             <state_interface name="velocity" />
         </joint>
-        <joint name="rear_left_wheel_joint">
+        <joint name="rear_right_wheel_joint">
             <command_interface name="velocity">
-              <param name="min">-1</param>
-              <param name="max">1</param>
+              <param name="min">-10</param>
+              <param name="max">10</param>
             </command_interface>
             <state_interface name="position" />
             <state_interface name="velocity" />
         </joint>
-        <joint name="front_right_wheel_joint">
-            <command_interface name="velocity">
-              <param name="min">-1</param>
-              <param name="max">1</param>
-            </command_interface>
-            <state_interface name="position" />
-            <state_interface name="velocity" />
-        </joint>
-        <joint name="front_left_wheel_joint">
-            <command_interface name="velocity">
-              <param name="min">-1</param>
-              <param name="max">1</param>
-            </command_interface>
-            <state_interface name="position" />
-            <state_interface name="velocity" />
-        </joint>
+        <xacro:if value="$(arg use_sim)">
+            <joint name="front_left_wheel_joint">
+                <command_interface name="velocity">
+                  <param name="min">-10</param>
+                  <param name="max">10</param>
+                </command_interface>
+                <state_interface name="position" />
+                <state_interface name="velocity" />
+            </joint>
+            <joint name="front_right_wheel_joint">
+                <command_interface name="velocity">
+                  <param name="min">-10</param>
+                  <param name="max">10</param>
+                </command_interface>
+                <state_interface name="position" />
+                <state_interface name="velocity" />
+            </joint>
+        </xacro:if>
     </ros2_control>
 </robot>
