Commit message: fix fortmat far bumperbot example

File: src/volcanibot_description/urdf/volcanibot.xacro (robot description, xacro)
@@ -1,9 +1,13 @@
-<?xml version="1.0" encoding="utf-8"?>
-<robot name="volcanibot_description" xmlns:xacro="http://www.ros.org/wiki/xacro">
+<?xml version="1.0"?>
+<robot xmlns:xacro="http://www.ros.org/wiki/xacro" name="volcanibot">
+  <!-- Gazebo plugins -->
+  <!-- <xacro:include filename="$(find volcanibot_description)/urdf/volcanibot.gazebo.xacro" /> -->
+  <!-- colors -->
+  <xacro:include filename="$(find volcanibot_description)/urdf/materials.xacro" />
   <!-- Define the world link -->
-  <link name="world"/>
+  <link name="base_footprint"/>
   <!-- Define a joint connecting world to base_link -->
-  <joint name="world_to_base_link" type="fixed">
-    <parent link="world"/>
+  <joint name="base_footprint_to_base_link" type="fixed">
+    <parent link="base_footprint"/>
     <child link="base_link"/>
     <origin xyz="0 0 0.9" rpy="0 0 0"/>
@@ -31,5 +35,5 @@
     </collision>
   </link>
-  <link name="link_BR">
+  <link name="rear_right_wheel_link">
     <inertial>
       <origin xyz="-0.002464 7.7174E-12 -1.0734E-12" rpy="0 0 0" />
@@ -40,5 +44,5 @@
       <origin xyz="0 0 0" rpy="0 0 0" />
       <geometry>
-        <mesh filename="package://volcanibot_description/meshes/link_BR.STL" />
+        <mesh filename="package://volcanibot_description/meshes/rear_right_wheel_link.STL" />
       </geometry>
       <material name="">
@@ -49,15 +53,15 @@
       <origin xyz="0 0 0" rpy="0 0 0" />
       <geometry>
-        <mesh filename="package://volcanibot_description/meshes/link_BR.STL" />
+        <mesh filename="package://volcanibot_description/meshes/rear_right_wheel_link.STL" />
       </geometry>
     </collision>
   </link>
-  <joint name="joint_BR" type="continuous">
+  <joint name="rear_right_wheel_joint" type="continuous">
     <origin xyz="0.9705 -0.5 -0.66" rpy="0 0 0" />
     <parent link="base_link" />
-    <child link="link_BR" />
+    <child link="rear_right_wheel_link" />
     <axis xyz="1 0 0" />
   </joint>
-  <link name="link_BL">
+  <link name="rear_left_wheel_link">
     <inertial>
       <origin xyz="0.002464 -4.863E-12 6.0718E-12" rpy="0 0 0" />
@@ -68,5 +72,5 @@
       <origin xyz="0 0 0" rpy="0 0 0" />
       <geometry>
-        <mesh filename="package://volcanibot_description/meshes/link_BL.STL" />
+        <mesh filename="package://volcanibot_description/meshes/rear_left_wheel_link.STL" />
       </geometry>
       <material name="">
@@ -77,15 +81,15 @@
       <origin xyz="0 0 0" rpy="0 0 0" />
       <geometry>
-        <mesh filename="package://volcanibot_description/meshes/link_BL.STL" />
+        <mesh filename="package://volcanibot_description/meshes/rear_left_wheel_link.STL" />
       </geometry>
     </collision>
   </link>
-  <joint name="joint_BL" type="continuous">
+  <joint name="rear_left_wheel_joint" type="continuous">
     <origin xyz="-0.9705 -0.5 -0.66" rpy="0 0 0" />
     <parent link="base_link" />
-    <child link="link_BL" />
+    <child link="rear_left_wheel_link" />
     <axis xyz="1 0 0" />
   </joint>
-  <link name="link_FL">
+  <link name="front_left_wheel_link">
     <inertial>
       <origin xyz="0.002464 3.0038E-12 7.1789E-12" rpy="0 0 0" />
@@ -96,5 +100,5 @@
       <origin xyz="0 0 0" rpy="0 0 0" />
       <geometry>
-        <mesh filename="package://volcanibot_description/meshes/link_FL.STL" />
+        <mesh filename="package://volcanibot_description/meshes/front_left_wheel_link.STL" />
       </geometry>
       <material name="">
@@ -105,15 +109,15 @@
       <origin xyz="0 0 0" rpy="0 0 0" />
       <geometry>
-        <mesh filename="package://volcanibot_description/meshes/link_FL.STL" />
+        <mesh filename="package://volcanibot_description/meshes/front_left_wheel_link.STL" />
       </geometry>
     </collision>
   </link>
-  <joint name="joint_FL" type="continuous">
+  <joint name="front_left_wheel_joint" type="continuous">
     <origin xyz="-0.9705 0.5 -0.66" rpy="0 0 0" />
     <parent link="base_link" />
-    <child link="link_FL" />
+    <child link="front_left_wheel_link" />
     <axis xyz="1 0 0" />
   </joint>
-  <link name="link_FR">
+  <link name="front_right_wheel_link">
     <inertial>
       <origin xyz="-0.002464 7.518E-12 2.0106E-12" rpy="0 0 0" />
@@ -124,5 +128,5 @@
       <origin xyz="0 0 0" rpy="0 0 0" />
       <geometry>
-        <mesh filename="package://volcanibot_description/meshes/link_FR.STL" />
+        <mesh filename="package://volcanibot_description/meshes/front_right_wheel_link.STL" />
       </geometry>
       <material name="">
@@ -133,12 +137,12 @@
       <origin xyz="0 0 0" rpy="0 0 0" />
       <geometry>
-        <mesh filename="package://volcanibot_description/meshes/link_FR.STL" />
+        <mesh filename="package://volcanibot_description/meshes/front_right_wheel_link.STL" />
       </geometry>
     </collision>
   </link>
-  <joint name="joint_FR" type="continuous">
+  <joint name="front_right_wheel_joint" type="continuous">
     <origin xyz="0.9705 0.5 -0.66" rpy="0 0 0" />
     <parent link="base_link" />
-    <child link="link_FR" />
+    <child link="front_right_wheel_link" />
     <axis xyz="1 0 0" />
   </joint>

Commit message: Fix cmd_vel delay bug when Gazebo start

File: src/volcanibot_description/urdf/volcanibot.xacro (robot description, xacro)
@@ -56,5 +56,5 @@
       <origin xyz="0 0 0" rpy="0 0 0" />
       <geometry>
-        <mesh filename="package://volcanibot_description/meshes/rear_right_wheel_link.STL" />
+        <sphere radius="0.26"/>
       </geometry>
     </collision>
@@ -84,5 +84,5 @@
       <origin xyz="0 0 0" rpy="0 0 0" />
       <geometry>
-        <mesh filename="package://volcanibot_description/meshes/rear_left_wheel_link.STL" />
+        <sphere radius="0.26"/>
       </geometry>
     </collision>
@@ -112,5 +112,5 @@
       <origin xyz="0 0 0" rpy="0 0 0" />
       <geometry>
-        <mesh filename="package://volcanibot_description/meshes/front_left_wheel_link.STL" />
+        <sphere radius="0.26"/>
       </geometry>
     </collision>
@@ -140,5 +140,5 @@
       <origin xyz="0 0 0" rpy="0 0 0" />
       <geometry>
-        <mesh filename="package://volcanibot_description/meshes/front_right_wheel_link.STL" />
+        <sphere radius="0.26"/>
       </geometry>
     </collision>

Commit message: Fix urdf file & STLs to align with the correct x axis

File: src/volcanibot_description/urdf/volcanibot.xacro (robot description, xacro)
@@ -18,7 +18,16 @@
   <link name="base_link">
     <inertial>
-      <origin xyz="-0.000308432013766069 0.000824745609093291 -0.348795097773964" rpy="0 0 0" />
-      <mass value="98.2206347258375" />
-      <inertia ixx="8.02628327825717" ixy="0.00024350529649604" ixz="2.67248679783338E-13" iyy="8.04861649065601" iyz="-1.25831921649467E-12" izz="14.6198876609904" />
+      <origin
+        xyz="0.000824745609091071 0.000308432013766069 -0.348795097773962"
+        rpy="0 0 0" />
+      <mass
+        value="98.2206347258376" />
+      <inertia
+        ixx="8.04861649065602"
+        ixy="-0.000243505296496384"
+        ixz="-1.23536316318022E-12"
+        iyy="8.02628327825716"
+        iyz="-2.67210376330799E-13"
+        izz="14.6198876609904" />
     </inertial>
     <visual>
@@ -27,7 +36,5 @@
         <mesh filename="package://volcanibot_description/meshes/base_link.STL" />
       </geometry>
-      <material name="">
-        <color rgba="0.792156862745098 0.819607843137255 0.933333333333333 1" />
-      </material>
+      <material name="red"/>
     </visual>
     <collision>
@@ -40,7 +47,16 @@
   <link name="rear_right_wheel_link">
     <inertial>
-      <origin xyz="-0.002464 7.7174E-12 -1.0734E-12" rpy="0 0 0" />
-      <mass value="19.568" />
-      <inertia ixx="0.76858" ixy="-1.5351E-12" ixz="4.2467E-13" iyy="0.41546" iyz="-7.8249E-13" izz="0.41546" />
+      <origin
+        xyz="7.66942065411058E-12 0.00246396479612621 -1.02851061001275E-12"
+        rpy="0 0 0" />
+      <mass
+        value="19.5682646733117" />
+      <inertia
+        ixx="0.41545797245674"
+        ixy="1.5364211917504E-12"
+        ixz="-7.82486812116746E-13"
+        iyy="0.768576636338704"
+        iyz="-4.25891260535319E-13"
+        izz="0.415457972457063" />
     </inertial>
     <visual>
@@ -49,7 +65,5 @@
         <mesh filename="package://volcanibot_description/meshes/rear_right_wheel_link.STL" />
       </geometry>
-      <material name="">
-        <color rgba="0.79216 0.81961 0.93333 1" />
-      </material>
+      <material name="black"/>
     </visual>
     <collision>
@@ -61,14 +75,28 @@
   </link>
   <joint name="rear_right_wheel_joint" type="continuous">
-    <origin xyz="0.9705 -0.5 -0.66" rpy="0 0 0" />
-    <parent link="base_link" />
-    <child link="rear_right_wheel_link" />
-    <axis xyz="1 0 0" />
+    <origin
+      xyz="-0.5 -0.9705 -0.66"
+      rpy="0 0 0" />
+    <parent
+      link="base_link" />
+    <child
+      link="rear_right_wheel_link" />
+    <axis
+      xyz="0 1 0" />
   </joint>
   <link name="rear_left_wheel_link">
     <inertial>
-      <origin xyz="0.002464 -4.863E-12 6.0718E-12" rpy="0 0 0" />
-      <mass value="19.568" />
-      <inertia ixx="0.76858" ixy="-1.1522E-12" ixz="1.0999E-12" iyy="0.41546" iyz="-2.2866E-13" izz="0.41546" />
+      <origin
+        xyz="-4.86310991476557E-12 -0.00246396479612798 6.07225381088483E-12"
+        rpy="0 0 0" />
+      <mass
+        value="19.568264673306" />
+      <inertia
+        ixx="0.415457972457667"
+        ixy="1.15340457833747E-12"
+        ixz="-2.28669379319239E-13"
+        iyy="0.768576636338705"
+        iyz="-1.1012630858852E-12"
+        izz="0.415457972456137" />
     </inertial>
     <visual>
@@ -77,7 +105,5 @@
         <mesh filename="package://volcanibot_description/meshes/rear_left_wheel_link.STL" />
       </geometry>
-      <material name="">
-        <color rgba="0.79216 0.81961 0.93333 1" />
-      </material>
+      <material name="black"/>
     </visual>
     <collision>
@@ -89,14 +115,28 @@
   </link>
   <joint name="rear_left_wheel_joint" type="continuous">
-    <origin xyz="-0.9705 -0.5 -0.66" rpy="0 0 0" />
-    <parent link="base_link" />
-    <child link="rear_left_wheel_link" />
-    <axis xyz="1 0 0" />
+    <origin
+      xyz="-0.5 0.9705 -0.66"
+      rpy="0 0 0" />
+    <parent
+      link="base_link" />
+    <child
+      link="rear_left_wheel_link" />
+    <axis
+      xyz="0 1 0" />
   </joint>
   <link name="front_left_wheel_link">
     <inertial>
-      <origin xyz="0.002464 3.0038E-12 7.1789E-12" rpy="0 0 0" />
-      <mass value="19.568" />
-      <inertia ixx="0.76858" ixy="4.1738E-13" ixz="1.5377E-12" iyy="0.41546" iyz="-5.1651E-13" izz="0.41546" />
+      <origin
+        xyz="3.00337532621597E-12 -0.00246396479612554 7.17892412183119E-12"
+        rpy="0 0 0" />
+      <mass
+        value="19.5682646733116" />
+      <inertia
+        ixx="0.415457972456292"
+        ixy="-4.16150298831959E-13"
+        ixz="-5.16513213527462E-13"
+        iyy="0.768576636338703"
+        iyz="-1.53906128365951E-12"
+        izz="0.415457972457511" />
     </inertial>
     <visual>
@@ -105,7 +145,5 @@
         <mesh filename="package://volcanibot_description/meshes/front_left_wheel_link.STL" />
       </geometry>
-      <material name="">
-        <color rgba="0.79216 0.81961 0.93333 1" />
-      </material>
+      <material name="black"/>
     </visual>
     <collision>
@@ -117,14 +155,28 @@
   </link>
   <joint name="front_left_wheel_joint" type="continuous">
-    <origin xyz="-0.9705 0.5 -0.66" rpy="0 0 0" />
-    <parent link="base_link" />
-    <child link="front_left_wheel_link" />
-    <axis xyz="1 0 0" />
+    <origin
+      xyz="0.5 0.9705 -0.66"
+      rpy="0 0 0" />
+    <parent
+      link="base_link" />
+    <child
+      link="front_left_wheel_link" />
+    <axis
+      xyz="0 1 0" />
   </joint>
   <link name="front_right_wheel_link">
     <inertial>
-      <origin xyz="-0.002464 7.518E-12 2.0106E-12" rpy="0 0 0" />
-      <mass value="19.568" />
-      <inertia ixx="0.76858" ixy="-1.5806E-12" ixz="-2.0336E-13" iyy="0.41546" iyz="-6.6262E-13" izz="0.41546" />
+      <origin
+        xyz="7.52264917025514E-12 0.00246396479612709 1.99529281985633E-12"
+        rpy="0 0 0" />
+      <mass
+        value="19.5682646733087" />
+      <inertia
+        ixx="0.415457972457348"
+        ixy="1.58185015757493E-12"
+        ixz="-6.62619227143719E-13"
+        iyy="0.768576636338703"
+        iyz="2.0216381958391E-13"
+        izz="0.415457972456455" />
     </inertial>
     <visual>
@@ -133,7 +185,5 @@
         <mesh filename="package://volcanibot_description/meshes/front_right_wheel_link.STL" />
       </geometry>
-      <material name="">
-        <color rgba="0.79216 0.81961 0.93333 1" />
-      </material>
+      <material name="black"/>
     </visual>
     <collision>
@@ -145,8 +195,13 @@
   </link>
   <joint name="front_right_wheel_joint" type="continuous">
-    <origin xyz="0.9705 0.5 -0.66" rpy="0 0 0" />
-    <parent link="base_link" />
-    <child link="front_right_wheel_link" />
-    <axis xyz="1 0 0" />
+    <origin
+      xyz="0.5 -0.9705 -0.66"
+      rpy="0 0 0" />
+    <parent
+      link="base_link" />
+    <child
+      link="front_right_wheel_link" />
+    <axis
+      xyz="0 1 0" />
   </joint>
 </robot>

Commit message: Add rgbd camera gazebo tags

File: src/volcanibot_description/urdf/volcanibot.xacro (robot description, xacro)
@@ -205,3 +205,44 @@
       xyz="0 1 0" />
   </joint>
+  <!-- Depth Camera -->
+  <joint type="fixed" name="camera_joint">
+    <origin xyz="0.225 0 0.075" rpy="0 0 0"/>
+    <child link="camera_link"/>
+    <parent link="base_link"/>
+    <axis xyz="0 1 0" />
+  </joint>
+  <link name='camera_link'>
+    <pose>0 0 0 0 0 0</pose>
+    <inertial>
+      <mass value="0.1"/>
+      <origin xyz="0 0 0" rpy="0 0 0"/>
+      <inertia
+          ixx="1e-6" ixy="0" ixz="0"
+          iyy="1e-6" iyz="0"
+          izz="1e-6"
+      />
+    </inertial>
+    <collision name='collision'>
+      <origin xyz="0 0 0" rpy="0 0 0"/>
+      <geometry>
+        <box size=".03 .03 .03"/>
+      </geometry>
+    </collision>
+    <visual name='camera_link_visual'>
+      <origin xyz="0 0 0" rpy="0 0 0"/>
+      <geometry>
+        <box size=".03 .03 .03"/>
+      </geometry>
+    </visual>
+  </link>
+  <gazebo reference="camera_link">
+    <material>Gazebo/Red</material>
+  </gazebo>
+  <joint type="fixed" name="camera_optical_joint">
+    <origin xyz="0 0 0" rpy="-1.5707 0 -1.5707"/>
+    <child link="camera_link_optical"/>
+    <parent link="camera_link"/>
+  </joint>
+  <link name="camera_link_optical">
+  </link>
 </robot>

File: src/volcanibot_description/urdf/volcanibot_gazebo.xacro (robot description, xacro)
@@ -53,3 +53,24 @@
     </xacro:unless>
   </gazebo>
+    <gazebo reference="camera_link">
+    <sensor name="rgbd_camera" type="rgbd_camera">
+      <camera>
+        <horizontal_fov>1.25</horizontal_fov>
+        <image>
+          <width>320</width>
+          <height>240</height>
+        </image>
+        <clip>
+          <near>0.3</near>
+          <far>15</far>
+        </clip>
+        <optical_frame_id>camera_link_optical</optical_frame_id>
+      </camera>
+      <always_on>1</always_on>
+      <update_rate>20</update_rate>
+      <visualize>true</visualize>
+      <topic>camera</topic>
+      <gz_frame_id>camera_link</gz_frame_id>
+    </sensor>
+  </gazebo>
 </robot>

Commit message: Add RViz configuration and RGBD camera URDF model
- Created a new RViz configuration file to set up visualization parameters for the robot model, camera, and depth cloud.
- Added a detailed URDF model for the RGBD camera, including joints, links, and Gazebo sensor configuration.

File: src/volcanibot_description/urdf/volcanibot.xacro (robot description, xacro)
@@ -2,4 +2,5 @@
 <robot xmlns:xacro="http://www.ros.org/wiki/xacro" name="volcanibot">
   <xacro:arg name="is_ignition" default="true" />
+  <xacro:arg name="prefix" default=""/>
   <!-- Include Gazebo plugins -->
   <xacro:include filename="$(find volcanibot_description)/urdf/volcanibot_gazebo.xacro" />
@@ -8,12 +9,8 @@
   <!-- Colors -->
   <xacro:include filename="$(find volcanibot_description)/urdf/materials.xacro" />
+  <!-- rgbd camera -->
+  <xacro:include filename="$(find volcanibot_description)/urdf/sensors/rgbd_camera.urdf.xacro" />
   <!-- Define the world link -->
   <link name="base_footprint"/>
-  <!-- Define a joint connecting world to base_link -->
-  <joint name="base_footprint_to_base_link" type="fixed">
-    <parent link="base_footprint"/>
-    <child link="base_link"/>
-    <origin xyz="0 0 0.9" rpy="0 0 0"/>
-  </joint>
   <link name="base_link">
     <inertial>
@@ -45,4 +42,10 @@
     </collision>
   </link>
+  <!-- Define a joint connecting world to base_link -->
+  <joint name="base_footprint_to_base_link" type="fixed">
+    <parent link="base_footprint"/>
+    <child link="base_link"/>
+    <origin xyz="0 0 0.9" rpy="0 0 0"/>
+  </joint>
   <link name="rear_right_wheel_link">
     <inertial>
@@ -206,5 +209,5 @@
   </joint>
   <!-- Depth Camera -->
-  <joint type="fixed" name="camera_joint">
+  <!-- <joint type="fixed" name="camera_joint">
     <origin xyz="0.225 0 0.075" rpy="0 0 0"/>
     <child link="camera_link"/>
@@ -245,4 +248,66 @@
   </joint>
   <link name="camera_link_optical">
-  </link>
+  </link> -->
+  <!-- Define the camera link -->
+  <!-- <link name="${prefix}rgbd_camera_link">
+    <visual>
+      <origin xyz="0 0 0" rpy="0 0 0"/>
+      <geometry>
+        <mesh filename="${mesh_file}" xyz="${mesh_xyz_offset}" rpy="${mesh_rpy_offset}"/>
+      </geometry>
+      <material name="red"/>
+    </visual>
+    <xacro:if value="${enable_collision}">
+      <collision>
+        <origin xyz="${collision_xyz_offset}" rpy="${collision_rpy_offset}"/>
+        <geometry>
+          <box size="${cam_depth} ${cam_width} ${cam_height}"/>
+        </geometry>
+      </collision>
+    </xacro:if>
+    <inertial>
+      <mass value="${mass}" />
+      <origin xyz="${inertial_xyz_offset}" rpy="${inertial_rpy_offset}"/>
+      <inertia ixx="${ixx}" ixy="${ixy}" ixz="${ixz}"
+               iyy="${iyy}" iyz="${iyz}" izz="${izz}" />
+    </inertial>
+  </link>
+  <joint name="${prefix}rgbd_camera_joint" type="fixed">
+    <parent link="${prefix}${parent}"/>
+    <child link="${prefix}rgbd_camera_link"/>
+    <origin xyz="${xyz_offset}" rpy="${rpy_offset}"/>
+  </joint> -->
+  <!-- Camera Link-->
+  <link name="rgbd_camera_link">
+      <inertial>
+          <mass value="0.001"/>
+          <origin rpy="0 0 0" xyz="0 0 0"/>
+          <inertia ixx="0.0001" ixy="0" ixz="0" iyy="0.0001" iyz="0" izz="0.0001"/>
+      </inertial>
+      <visual>
+          <origin rpy="0 0 0" xyz="0 0 0"/>
+          <geometry>
+              <sphere radius="0.001"/>
+          </geometry>
+          <material name="">
+              <color rgba="0.5 0 0 1" />
+          </material>
+      </visual>
+      <collision>
+          <origin rpy="0 0 0" xyz="0 0 0"/>
+          <geometry>
+              <sphere radius="0.001"/>
+          </geometry>
+      </collision>
+  </link>
+  <joint name="rgbd_camera_joint" type="fixed">
+      <parent link="base_link"/>
+      <child link="rgbd_camera_link"/>
+      <origin rpy="0 0 0" xyz="0.225 0 0.075"/>
+  </joint>
+  <!-- rgbd camera -->
+  <xacro:rgbd_camera
+    camera_name="realsense_d435"
+    xyz_offset="0.225 0 0.075"
+  />
 </robot>

File: src/volcanibot_description/urdf/volcanibot_gazebo.xacro (robot description, xacro)
@@ -53,5 +53,5 @@
     </xacro:unless>
   </gazebo>
-    <gazebo reference="camera_link">
+    <!-- <gazebo reference="camera_link">
     <sensor name="rgbd_camera" type="rgbd_camera">
       <camera>
@@ -73,4 +73,4 @@
       <gz_frame_id>camera_link</gz_frame_id>
     </sensor>
-  </gazebo>
+  </gazebo>  -->
 </robot>
