Commit message: Revert "Add RViz configuration and RGBD camera URDF model"

File: src/volcanibot_description/urdf/volcanibot.xacro (robot description, xacro)
@@ -2,5 +2,4 @@
 <robot xmlns:xacro="http://www.ros.org/wiki/xacro" name="volcanibot">
   <xacro:arg name="is_ignition" default="true" />
-  <xacro:arg name="prefix" default=""/>
   <!-- Include Gazebo plugins -->
   <xacro:include filename="$(find volcanibot_description)/urdf/volcanibot_gazebo.xacro" />
@@ -9,8 +8,12 @@
   <!-- Colors -->
   <xacro:include filename="$(find volcanibot_description)/urdf/materials.xacro" />
-  <!-- rgbd camera -->
-  <xacro:include filename="$(find volcanibot_description)/urdf/sensors/rgbd_camera.urdf.xacro" />
   <!-- Define the world link -->
   <link name="base_footprint"/>
+  <!-- Define a joint connecting world to base_link -->
+  <joint name="base_footprint_to_base_link" type="fixed">
+    <parent link="base_footprint"/>
+    <child link="base_link"/>
+    <origin xyz="0 0 0.9" rpy="0 0 0"/>
+  </joint>
   <link name="base_link">
     <inertial>
@@ -42,10 +45,4 @@
     </collision>
   </link>
-  <!-- Define a joint connecting world to base_link -->
-  <joint name="base_footprint_to_base_link" type="fixed">
-    <parent link="base_footprint"/>
-    <child link="base_link"/>
-    <origin xyz="0 0 0.9" rpy="0 0 0"/>
-  </joint>
   <link name="rear_right_wheel_link">
     <inertial>
@@ -209,5 +206,5 @@
   </joint>
   <!-- Depth Camera -->
-  <!-- <joint type="fixed" name="camera_joint">
+  <joint type="fixed" name="camera_joint">
     <origin xyz="0.225 0 0.075" rpy="0 0 0"/>
     <child link="camera_link"/>
@@ -248,66 +245,4 @@
   </joint>
   <link name="camera_link_optical">
-  </link> -->
-  <!-- Define the camera link -->
-  <!-- <link name="${prefix}rgbd_camera_link">
-    <visual>
-      <origin xyz="0 0 0" rpy="0 0 0"/>
-      <geometry>
-        <mesh filename="${mesh_file}" xyz="${mesh_xyz_offset}" rpy="${mesh_rpy_offset}"/>
-      </geometry>
-      <material name="red"/>
-    </visual>
-    <xacro:if value="${enable_collision}">
-      <collision>
-        <origin xyz="${collision_xyz_offset}" rpy="${collision_rpy_offset}"/>
-        <geometry>
-          <box size="${cam_depth} ${cam_width} ${cam_height}"/>
-        </geometry>
-      </collision>
-    </xacro:if>
-    <inertial>
-      <mass value="${mass}" />
-      <origin xyz="${inertial_xyz_offset}" rpy="${inertial_rpy_offset}"/>
-      <inertia ixx="${ixx}" ixy="${ixy}" ixz="${ixz}"
-               iyy="${iyy}" iyz="${iyz}" izz="${izz}" />
-    </inertial>
-  </link>
-  <joint name="${prefix}rgbd_camera_joint" type="fixed">
-    <parent link="${prefix}${parent}"/>
-    <child link="${prefix}rgbd_camera_link"/>
-    <origin xyz="${xyz_offset}" rpy="${rpy_offset}"/>
-  </joint> -->
-  <!-- Camera Link-->
-  <link name="rgbd_camera_link">
-      <inertial>
-          <mass value="0.001"/>
-          <origin rpy="0 0 0" xyz="0 0 0"/>
-          <inertia ixx="0.0001" ixy="0" ixz="0" iyy="0.0001" iyz="0" izz="0.0001"/>
-      </inertial>
-      <visual>
-          <origin rpy="0 0 0" xyz="0 0 0"/>
-          <geometry>
-              <sphere radius="0.001"/>
-          </geometry>
-          <material name="">
-              <color rgba="0.5 0 0 1" />
-          </material>
-      </visual>
-      <collision>
-          <origin rpy="0 0 0" xyz="0 0 0"/>
-          <geometry>
-              <sphere radius="0.001"/>
-          </geometry>
-      </collision>
-  </link>
-  <joint name="rgbd_camera_joint" type="fixed">
-      <parent link="base_link"/>
-      <child link="rgbd_camera_link"/>
-      <origin rpy="0 0 0" xyz="0.225 0 0.075"/>
-  </joint>
-  <!-- rgbd camera -->
-  <xacro:rgbd_camera
-    camera_name="realsense_d435"
-    xyz_offset="0.225 0 0.075"
-  />
+  </link>
 </robot>

File: src/volcanibot_description/urdf/volcanibot_gazebo.xacro (robot description, xacro)
@@ -53,5 +53,5 @@
     </xacro:unless>
   </gazebo>
-    <!-- <gazebo reference="camera_link">
+    <gazebo reference="camera_link">
     <sensor name="rgbd_camera" type="rgbd_camera">
       <camera>
@@ -73,4 +73,4 @@
       <gz_frame_id>camera_link</gz_frame_id>
     </sensor>
-  </gazebo>  -->
+  </gazebo>
 </robot>

Commit message: Add rgbd camera

File: src/volcanibot_description/urdf/volcanibot.xacro (robot description, xacro)
@@ -205,3 +205,44 @@
       xyz="0 1 0" />
   </joint>
+    <!-- Depth Camera -->
+  <joint type="fixed" name="camera_joint">
+    <origin xyz="0.6 0 0.07" rpy="0 0.2 0"/>
+    <child link="camera_link"/>
+    <parent link="base_link"/>
+    <axis xyz="0 1 0" />
+  </joint>
+  <link name='camera_link'>
+    <pose>0 0 0 0 0 0</pose>
+    <inertial>
+      <mass value="0.1"/>
+      <origin xyz="0 0 0" rpy="0 0 0"/>
+      <inertia
+          ixx="1e-6" ixy="0" ixz="0"
+          iyy="1e-6" iyz="0"
+          izz="1e-6"
+      />
+    </inertial>
+    <collision name='collision'>
+      <origin xyz="0 0 0" rpy="0 0 0"/>
+      <geometry>
+         <box size=".03 .03 .03"/>
+      </geometry>
+    </collision>
+    <visual name='camera_link_visual'>
+      <origin xyz="0 0 0" rpy="0 0 0"/>
+      <geometry>
+        <box size=".03 .03 .03"/>
+      </geometry>
+    </visual>
+  </link>
+  <gazebo reference="camera_link">
+    <material>Gazebo/Red</material>
+  </gazebo>
+  <joint type="fixed" name="camera_optical_joint">
+    <origin xyz="0 0 0" rpy="-1.5707 0 -1.5707"/>
+    <child link="camera_link_optical"/>
+    <parent link="camera_link"/>
+  </joint>
+  <link name="camera_link_optical">
+  </link>
 </robot>

File: src/volcanibot_description/urdf/volcanibot_gazebo.xacro (robot description, xacro)
@@ -53,3 +53,24 @@
     </xacro:unless>
   </gazebo>
+  <gazebo reference="camera_link">
+    <sensor name="rgbd_camera" type="rgbd_camera">
+      <camera>
+        <horizontal_fov>1.25</horizontal_fov>
+        <image>
+          <width>320</width>
+          <height>240</height>
+        </image>
+        <clip>
+          <near>0.3</near>
+          <far>15</far>
+        </clip>
+        <optical_frame_id>camera_link_optical</optical_frame_id>
+      </camera>
+      <always_on>1</always_on>
+      <update_rate>20</update_rate>
+      <visualize>true</visualize>
+      <topic>camera</topic>
+      <gz_frame_id>camera_link</gz_frame_id>
+    </sensor>
+  </gazebo>
 </robot>

Commit message: Tune joystick teleop and add real-robot front-wheel mimic joints
- Lower joy deadzone 0.5->0.1 for finer stick response
- Adjust teleop scales: linear-x 1.0->2.0, angular-z 8.0->1.7
- Mimic front wheels off rear joints on real hardware (unactuated,
  chained); sim continues to drive all 4 wheels directly

File: src/volcanibot_description/urdf/volcanibot.xacro (robot description, xacro)
@@ -173,4 +173,10 @@
     <axis
       xyz="0 1 0" />
+    <!-- Real robot: front wheel is chained to the rear and has no actuator.
+         Mimic lets robot_state_publisher derive its TF from the rear joint.
+         Sim drives all 4 wheels directly (gz physics ignores mimic). -->
+    <xacro:unless value="$(arg use_sim)">
+      <mimic joint="rear_left_wheel_joint" multiplier="1.0" offset="0.0"/>
+    </xacro:unless>
   </joint>
   <link name="front_right_wheel_link">
@@ -213,4 +219,7 @@
     <axis
       xyz="0 1 0" />
+    <xacro:unless value="$(arg use_sim)">
+      <mimic joint="rear_right_wheel_joint" multiplier="1.0" offset="0.0"/>
+    </xacro:unless>
   </joint>
   <!-- Optional RGBD camera -->

Commit message: Add optional Trimble RTK GPS (gps:=true) via vcstool + navsat
GPS is third-party, so the driver is pulled via volcanibot.repos pinned to
trimble-oss @ 613dca0 -- the last commit using the gsof_msgs/trimble_driver_ros
package names that gps.launch.py references (newer upstream renamed them).
Off by default; was WIP/commented-out in omribu's stack.

- gps.launch.py: gsof_client_node + navsat_transform_node, gated by gps:=true
- config/gsof_client_params.yaml (receiver ip/port) + navsat_params.yaml
- volcanibot.xacro: gps:=true adds dual GPS antenna links (+ GPS_Antenna.STL)
- real_bringup: gps arg -> xacro + gps.launch.py include
- trimble_driver_ros + robot_localization exec_depends

Building the driver needs apt deps (libgeographiclib-dev, libpcap0.8-dev,
boost) via rosdep -- verified resolvable. URDF gps path and launches validated.

File: src/volcanibot_description/urdf/volcanibot.xacro (robot description, xacro)
@@ -5,4 +5,5 @@
   <xacro:arg name="lidar" default="false" />
   <xacro:arg name="camera" default="false" />
+  <xacro:arg name="gps" default="false" />
   <xacro:arg name="serial_port" default="/dev/roboteq" />
   <xacro:arg name="baud_rate" default="115200" />
@@ -265,3 +266,57 @@
     </link>
   </xacro:if>
+  <!-- Optional dual GPS/RTK antennas (Trimble). Physical payload; included
+       only when gps:=true so sim and lidar/camera-only runs stay uncluttered. -->
+  <xacro:if value="$(arg gps)">
+    <link name="gps_antenna_pos_right">
+      <visual>
+        <origin xyz="-0.074 0.075 0" rpy="1.57 0 0"/>
+        <geometry>
+          <mesh filename="package://volcanibot_description/meshes/GPS_Antenna.STL" scale="0.001 0.001 0.001"/>
+        </geometry>
+        <material name="gps_silver">
+          <color rgba="0.75 0.75 0.78 1"/>
+        </material>
+      </visual>
+      <visual>
+        <origin xyz="0 0 -0.555" rpy="0 0 0"/>
+        <geometry>
+          <box size="0.02 0.02 1.11"/>
+        </geometry>
+        <material name="gps_rod">
+          <color rgba="0.5 0.5 0.52 1"/>
+        </material>
+      </visual>
+    </link>
+    <joint name="gps_antenna_pos_right_joint" type="fixed">
+      <parent link="base_link"/>
+      <child link="gps_antenna_pos_right"/>
+      <origin xyz="-0.6 -0.87 0.97" rpy="0 0 0"/>
+    </joint>
+    <link name="gps_antenna_pos_left">
+      <visual>
+        <origin xyz="-0.074 0.075 0" rpy="1.57 0 0"/>
+        <geometry>
+          <mesh filename="package://volcanibot_description/meshes/GPS_Antenna.STL" scale="0.001 0.001 0.001"/>
+        </geometry>
+        <material name="gps_silver">
+          <color rgba="0.75 0.75 0.78 1"/>
+        </material>
+      </visual>
+      <visual>
+        <origin xyz="0 0 -0.555" rpy="0 0 0"/>
+        <geometry>
+          <box size="0.02 0.02 1.11"/>
+        </geometry>
+        <material name="gps_rod">
+          <color rgba="0.5 0.5 0.52 1"/>
+        </material>
+      </visual>
+    </link>
+    <joint name="gps_antenna_pos_left_joint" type="fixed">
+      <parent link="base_link"/>
+      <child link="gps_antenna_pos_left"/>
+      <origin xyz="0.6 0.87 0.97" rpy="0 0 0"/>
+    </joint>
+  </xacro:if>
 </robot>

Commit message: Unify sim and real controller config; tune real-robot drive
Sim is now rear-driven like the real robot, so both share one config:
- front wheels follow the rear as URDF mimic joints (always on); in sim
  gz_ros2_control spins them, on the real robot they are mechanically chained
- sim ros2_control declares the front wheels as state-only mimic joints
- single volcanibot_controllers.yaml (rear-only, 50 Hz); drop the _real variant
  and point real_bringup at it

Real-robot drive fixes from comparing against the prior working setup:
- gear_ratio 1.0 -> 10.0 (10:1 motor:wheel reduction; was commanding a tenth of
  the motor RPM, hence the crawl)
- left_encoder_sign -> -1.0 (left motor mirror-mounted; odom read a turn while
  driving straight)
- limits 2.0 m/s / 1.7 rad/s, acceleration 1.0

File: src/volcanibot_description/urdf/volcanibot.xacro (robot description, xacro)
@@ -174,10 +174,9 @@
     <axis
       xyz="0 1 0" />
-    <!-- Real robot: front wheel is chained to the rear and has no actuator.
-         Mimic lets robot_state_publisher derive its TF from the rear joint.
-         Sim drives all 4 wheels directly (gz physics ignores mimic). -->
-    <xacro:unless value="$(arg use_sim)">
-      <mimic joint="rear_left_wheel_joint" multiplier="1.0" offset="0.0"/>
-    </xacro:unless>
+    <!-- Front wheel is chained to the rear with no actuator of its own, so it
+         mimics the rear joint. On the real robot this lets robot_state_publisher
+         derive the front TF; in sim gz_ros2_control drives the front wheel off
+         the rear so the robot is rear-driven like the real one. -->
+    <mimic joint="rear_left_wheel_joint" multiplier="1.0" offset="0.0"/>
   </joint>
   <link name="front_right_wheel_link">
@@ -220,7 +219,5 @@
     <axis
       xyz="0 1 0" />
-    <xacro:unless value="$(arg use_sim)">
-      <mimic joint="rear_right_wheel_joint" multiplier="1.0" offset="0.0"/>
-    </xacro:unless>
+    <mimic joint="rear_right_wheel_joint" multiplier="1.0" offset="0.0"/>
   </joint>
   <!-- Optional RGBD camera -->

File: src/volcanibot_description/urdf/volcanibot_ros2_control.xacro (robot description, xacro)
@@ -18,5 +18,5 @@
                 <param name="baud_rate">$(arg baud_rate)</param>
                 <param name="timeout_ms">1000</param>
-                <param name="gear_ratio">1.0</param>
+                <param name="gear_ratio">10.0</param>
                 <!-- Encoder counts per WHEEL revolution (encoder PPR x quadrature
                      x gear). CALIBRATE: roll a wheel exactly one turn and read
@@ -24,5 +24,5 @@
                      wheel drives forward. -->
                 <param name="counts_per_rev">10024.0</param>
-                <param name="left_encoder_sign">-1.0</param>
+                <param name="left_encoder_sign">-1.0</param>   <!-- left motor mirror-mounted: counts invert for forward -->
                 <param name="right_encoder_sign">1.0</param>
                 <param name="left_wheel_name">rear_left_wheel_joint</param>
@@ -30,9 +30,9 @@
             </xacro:unless>
         </hardware>
-        <!-- In sim, all 4 wheels are independently controlled by Gazebo (the
-             physics engine doesn't support URDF mimic joints). On the real
-             robot only the rear wheels are motorized; the front wheels are
-             mechanically chained to the rear and so are not exposed to
-             ros2_control. -->
+        <!-- Both sim and real are rear-driven (same controllers config). The
+             front wheels are chained to the rear: on the real robot they have no
+             actuator and aren't exposed to ros2_control; in sim they are
+             declared below as state-only mimic joints so gz_ros2_control spins
+             them off the rear (the URDF <mimic> tags drive the constraint). -->
         <joint name="rear_left_wheel_joint">
             <command_interface name="velocity">
@@ -51,18 +51,12 @@
             <state_interface name="velocity" />
         </joint>
+        <!-- Mimic joints: no command interface (driven by the URDF <mimic>
+             constraint off the rear wheels), state-only so they publish. -->
         <xacro:if value="$(arg use_sim)">
             <joint name="front_left_wheel_joint">
-                <command_interface name="velocity">
-                  <param name="min">-10</param>
-                  <param name="max">10</param>
-                </command_interface>
                 <state_interface name="position" />
                 <state_interface name="velocity" />
             </joint>
             <joint name="front_right_wheel_joint">
-                <command_interface name="velocity">
-                  <param name="min">-10</param>
-                  <param name="max">10</param>
-                </command_interface>
                 <state_interface name="position" />
                 <state_interface name="velocity" />
